Commit message: added kinect mount, disable collision

File: xarm_description/urdf/gripper/xarm_gripper.urdf.xacro (robot description, xacro)
@@ -5,8 +5,31 @@
       <joint name="${prefix}gripper_fix" type="fixed">
         <parent link="${attach_to}"/>
-        <child link="${prefix}xarm_gripper_base_link"/>
+        <child link="${prefix}kinect_mount"/>
         <origin xyz="${attach_xyz}" rpy="${attach_rpy}"/>
       </joint>
     </xacro:unless>
+    <link name="${prefix}kinect_mount">
+      <inertial>
+        <origin xyz="0 0 0" rpy="0 0 0" />
+        <mass value="0.52" />
+        <inertia
+          ixx="0.00020833" ixy="3.9292E-07" ixz="2.6537E-06"
+          iyy="0.00020833" iyz="-1.0975E-05" izz="0.00020833" />
+      </inertial>
+      <xacro:common_link_visual
+        mesh_filename="azure_kinect_mount"
+        origin_xyz="0.08 0 0.013"
+        origin_rpy="0 0 -1.5708"
+        material_name="${prefix}Silver" />
+      <xacro:common_link_collision
+        mesh_filename="azure_kinect_mount"
+        origin_xyz="0.08 0 0.013"
+        origin_rpy="0 0 -1.5708" />
+    </link>
+    <joint name="${prefix}kinect_joint" type="fixed">
+      <origin xyz="0 0 0.0125" rpy="0 0 0" />
+      <parent link="${prefix}kinect_mount" />
+      <child link="${prefix}xarm_gripper_base_link" />
+    </joint>
     <link name="${prefix}xarm_gripper_base_link">
       <inertial>

File: xarm_description/urdf/xarm6/xarm6_robot_macro.xacro (robot description, xacro)
@@ -35,5 +35,5 @@
           joint2_lower_limit="${-2.059}" joint2_upper_limit="${2.0944}"
           joint3_lower_limit="${-pi*0.99}" joint3_upper_limit="${0.19198}"
-          joint4_lower_limit="${-pi*0.99}" joint4_upper_limit="${pi*0.99}"
+          joint4_lower_limit="${-2*pi*0.99}" joint4_upper_limit="${2*pi*0.99}"
           joint5_lower_limit="${-1.69297}" joint5_upper_limit="${pi*0.99}"
           joint6_lower_limit="${-pi*0.99}" joint6_upper_limit="${pi*0.99}"/>
@@ -43,5 +43,5 @@
         joint2_lower_limit="${-2.059}" joint2_upper_limit="${2.0944}"
         joint3_lower_limit="${-pi*0.99}" joint3_upper_limit="${0.19198}"
-        joint4_lower_limit="${-pi*0.99}" joint4_upper_limit="${pi*0.99}"
+        joint4_lower_limit="${-2*pi*0.99}" joint4_upper_limit="${2*pi*0.99}"
         joint5_lower_limit="${-1.69297}" joint5_upper_limit="${pi*0.99}"
         joint6_lower_limit="${-pi*0.99}" joint6_upper_limit="${pi*0.99}"

File: xarm_moveit_config/srdf/_xarm6_macro.srdf.xacro (robot description, xacro)
@@ -54,4 +54,5 @@
     <xacro:if value="${add_gripper}">
       <group name="${prefix}xarm_gripper">
+        <link name="${prefix}kinect_mount" />
         <link name="${prefix}xarm_gripper_base_link" />
         <link name="${prefix}left_outer_knuckle" />
@@ -63,4 +64,5 @@
         <link name="${prefix}link_tcp" />
         <joint name="${prefix}drive_joint" />
+        <joint name="${prefix}kinect_joint" />
       </group>
       <group_state name="open" group="${prefix}xarm_gripper">
@@ -73,4 +75,5 @@
       <end_effector name="${prefix}xarm_gripper" parent_link="${prefix}link_tcp" group="${prefix}xarm_gripper" />
       <!--PASSIVE JOINT, Purpose, this element is used to mark joints that are not actuated-->
+      <passive_joint name="${prefix}kinect_joint" />
       <passive_joint name="${prefix}left_finger_joint" />
       <passive_joint name="${prefix}left_inner_knuckle_joint" />
@@ -125,5 +128,14 @@
       <disable_collisions link1="${prefix}link_eef" link2="${prefix}right_inner_knuckle" reason="Never" />
       <disable_collisions link1="${prefix}link_eef" link2="${prefix}right_outer_knuckle" reason="Never" />
-      <disable_collisions link1="${prefix}link_eef" link2="${prefix}xarm_gripper_base_link" reason="Adjacent" />
+      <disable_collisions link1="${prefix}link_eef" link2="${prefix}xarm_gripper_base_link" reason="Never" />
+      <disable_collisions link1="${prefix}link6" link2="${prefix}kinect_mount" reason="Never" />
+      <disable_collisions link1="${prefix}link_eef" link2="${prefix}kinect_mount" reason="Adjacent" />
+      <disable_collisions link1="${prefix}xarm_gripper_base_link" link2="${prefix}kinect_mount" reason="Adjacent" />
+      <disable_collisions link1="${prefix}left_finger" link2="${prefix}kinect_mount" reason="Never" />
+      <disable_collisions link1="${prefix}left_inner_knuckle" link2="${prefix}kinect_mount" reason="Never" />
+      <disable_collisions link1="${prefix}left_outer_knuckle" link2="${prefix}kinect_mount" reason="Never" />
+      <disable_collisions link1="${prefix}right_finger" link2="${prefix}kinect_mount" reason="Never" />
+      <disable_collisions link1="${prefix}right_inner_knuckle" link2="${prefix}kinect_mount" reason="Never" />
+      <disable_collisions link1="${prefix}right_outer_knuckle" link2="${prefix}kinect_mount" reason="Never" />
     </xacro:if>
     <!-- vacuum gripper -->
