Commit message: added linear direct motor base

File: xarm_description/urdf/xarm6/xarm6.urdf.xacro (robot description, xacro)
@@ -37,4 +37,28 @@
     </xacro:unless>
     <xacro:property name="kinematics_params" value="${kinematics_config['kinematics']}"/>
+    <link name="${prefix}linear_direct_motor_base">
+      <visual>
+        <origin xyz="0 -0.350 0" rpy="0 0 0" />
+        <geometry>
+          <box size="0.213 0.930 0.135" />
+        </geometry>
+        <material name="Blue">
+          <color rgba="0.28 0.52 0.92 1.0"/>
+        </material>
+      </visual>
+      <collision>
+        <origin xyz="0 -0.350 0" rpy="0 0 0" />
+        <geometry>
+          <box size="0.213 0.930 0.135"/>
+        </geometry>
+      </collision>
+    </link>
+    <joint name="${prefix}slider_joint" type="prismatic">
+        <parent link="${prefix}linear_direct_motor_base" />
+        <child link="${prefix}link_base" />
+        <origin xyz="0 0 0.0625" rpy="0 0 0" />
+        <axis xyz="0 -1 0" />
+        <limit lower="0" upper="0.7" velocity="1.0" effort="100"/>
+    </joint>
     <link name="${prefix}link_base">
       <inertial>

File: xarm_description/urdf/xarm_device_macro.xacro (robot description, xacro)
@@ -67,9 +67,18 @@
       <link name="world" />
     </xacro:if>
-    <joint name="${prefix}world_joint" type="fixed">
-      <parent link="${attach_to}" />
-      <child link="${prefix}link_base" />
-      <origin xyz="${attach_xyz}" rpy="${attach_rpy}" />
-    </joint>
+    <xacro:unless value="${robot_type == 'xarm' and dof == 6}">
+      <joint name="${prefix}world_joint" type="fixed">
+        <parent link="${attach_to}" />
+        <child link="${prefix}link_base" />
+        <origin xyz="${attach_xyz}" rpy="${attach_rpy}" />
+      </joint>
+    </xacro:unless>
+    <xacro:if value="${robot_type =='xarm' and dof == 6}">
+      <joint name="${prefix}world_joint" type="fixed">
+        <parent link="world" />
+        <child link="${prefix}linear_direct_motor_base" />
+        <origin xyz="0 0 0.0625" rpy="0 0 0" />
+      </joint>
+    </xacro:if>
     <xacro:if value="${effort_control}">
       <xacro:property name="hard_interface" value="EffortJointInterface" />

File: xarm_moveit_config/srdf/_xarm6_macro.srdf.xacro (robot description, xacro)
@@ -12,5 +12,4 @@
     add_gripper='false' add_vacuum_gripper='false' add_other_geometry='false' ">
     <group name="${prefix}xarm6">
-      <joint name="${prefix}world_joint" />
       <joint name="${prefix}joint1" />
       <joint name="${prefix}joint2" />
@@ -34,4 +33,8 @@
       </xacro:if>
     </group>
+    <group name="${prefix}slider">
+      <joint name="${prefix}slider_joint" />
+      <joint name="${prefix}world_joint" />
+    </group>
     <!-- GROUP STATES, Purpose, Define a named state for a particular group, in terms of joint values. This is useful to define states like 'folded arms' -->
     <group_state name="home" group="${prefix}xarm6">
@@ -51,4 +54,13 @@
       <joint name="${prefix}joint6" value="0" />
     </group_state>
+    <group_state name="centre" group="${prefix}xarm6">
+      <joint name="${prefix}joint1" value="1.41674" />
+      <joint name="${prefix}joint2" value="-0.6318" />
+      <joint name="${prefix}joint3" value="-0.24822" />
+      <joint name="${prefix}joint4" value="6.21608" />
+      <joint name="${prefix}joint5" value="0.8429123" />
+      <joint name="${prefix}joint6" value="-0.28200" />
+    </group_state>
+    <disable_collisions link1="${prefix}linear_direct_motor_base" link2="${prefix}link_base" reason="Adjacent" />
     <!-- gripper -->
     <xacro:if value="${add_gripper}">
